File: _autosave-korad_kel103_converter.kicad_pcb (KiCad board)
At the start: 2 copper layers, 47.9 x 44.9 mm, 6 parts, among them J1 Conn_01x01_Female, J2 Conn_01x01_Female, J3 Conn_01x01_Female, J4 Conn_01x01_Female, J5 Conn_01x01_Female, J6 Conn_01x01_Female

Commit message: Adding readme
Parts:
- J5, J6: footprint NetTie:NetTie-4_SMD_Pad2.0mm -> Local:SMD_pad_connector
- moved J6 7.87 mm to (126.3, 84.2), turned to 0 degrees
- moved J5 5.40 mm to (147.8, 78.8)
Routing:
- net Net-(J2-Pad1): vias 8 -> 23
- net Net-(J1-Pad1): vias 8 -> 23
Changed lines of the file:
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@@
     (thickness 1.6)
     (drawings 20)
-    (tracks 16)
+    (tracks 46)
     (zones 0)
     (modules 6)
@@
     (mod_text_size 1 1)
     (mod_text_width 0.15)
-    (pad_size 2 2)
-    (pad_drill 0.5)
+    (pad_size 8 4)
+    (pad_drill 0)
     (pad_to_mask_clearance 0)
     (aux_axis_origin 0 0)
@@
     (add_net "Net-(J2-Pad1)")
   )
-  (module NetTie:NetTie-4_SMD_Pad2.0mm (layer F.Cu)
-    (at 133 80 180)
-    (descr "Net tie, 4 pin, 2.0mm square SMD pads")
-    (tags "net tie")
-    (attr virtual)
-    (fp_text reference J6 (at 0 -4) (layer F.SilkS)
-      (effects (font (size 1 1) (thickness 0.15)))
-    )
-    (fp_text value Conn_01x01_Female (at 0 4) (layer F.Fab)
-      (effects (font (size 1 1) (thickness 0.15)))
-    )
-    (fp_poly (pts (xy -3 -3) (xy 3 -3) (xy 3 3) (xy -3 3)) (layer F.Cu) (width 0))
-    (fp_line (start -3.25 3.25) (end -3.25 -3.25) (layer F.CrtYd) (width 0.05))
-    (fp_line (start 3.25 3.25) (end -3.25 3.25) (layer F.CrtYd) (width 0.05))
-    (fp_line (start 3.25 -3.25) (end 3.25 3.25) (layer F.CrtYd) (width 0.05))
-    (fp_line (start -3.25 -3.25) (end 3.25 -3.25) (layer F.CrtYd) (width 0.05))
-    (pad 4 smd circle (at 2 2 180) (size 2 2) (layers F.Cu))
-    (pad 3 smd circle (at -2 2 180) (size 2 2) (layers F.Cu))
-    (pad 2 smd circle (at 2 -2 180) (size 2 2) (layers F.Cu))
-    (pad 1 smd circle (at -2 -2 180) (size 2 2) (layers F.Cu)
-      (net 1 "Net-(J1-Pad1)"))
-  )
-  (module NetTie:NetTie-4_SMD_Pad2.0mm (layer F.Cu)
-    (at 142.5 80 180)
-    (descr "Net tie, 4 pin, 2.0mm square SMD pads")
-    (tags "net tie")
-    (zone_connect 2)
-    (attr virtual)
-    (fp_text reference J5 (at 0 -4) (layer F.SilkS)
-      (effects (font (size 1 1) (thickness 0.15)))
-    )
-    (fp_text value Conn_01x01_Female (at 0 4) (layer F.Fab)
-      (effects (font (size 1 1) (thickness 0.15)))
-    )
-    (fp_poly (pts (xy -3 -3) (xy 3 -3) (xy 3 3) (xy -3 3)) (layer F.Cu) (width 0))
-    (fp_line (start -3.25 3.25) (end -3.25 -3.25) (layer F.CrtYd) (width 0.05))
-    (fp_line (start 3.25 3.25) (end -3.25 3.25) (layer F.CrtYd) (width 0.05))
-    (fp_line (start 3.25 -3.25) (end 3.25 3.25) (layer F.CrtYd) (width 0.05))
-    (fp_line (start -3.25 -3.25) (end 3.25 -3.25) (layer F.CrtYd) (width 0.05))
-    (pad 4 smd circle (at 2 2 180) (size 2 2) (layers F.Cu)
-      (zone_connect 2))
-    (pad 3 smd circle (at -2 2 180) (size 2 2) (layers F.Cu)
-      (zone_connect 2))
-    (pad 2 thru_hole circle (at 2 -2 180) (size 2 2) (drill 0.5) (layers *.Cu *.Mask)
-      (net 2 "Net-(J2-Pad1)") (zone_connect 2))
-    (pad 1 smd circle (at -2 -2 180) (size 2 2) (layers F.Cu)
-      (net 2 "Net-(J2-Pad1)") (zone_connect 2))
+  (module Local:SMD_pad_connector (layer F.Cu)
+    (at 126.35 84.2)
+    (fp_text reference J6 (at 0 0.5) (layer F.SilkS) hide
+      (effects (font (size 1 1) (thickness 0.15)))
+    )
+    (fp_text value Conn_01x01_Female (at 0 -0.5) (layer F.Fab) hide
+      (effects (font (size 1 1) (thickness 0.15)))
+    )
+    (pad 1 smd rect (at -0.1 -2.7) (size 8 4) (layers F.Cu F.Mask)
+      (net 1 "Net-(J1-Pad1)"))
+  )
+  (module Local:SMD_pad_connector (layer F.Cu)
+    (at 147.75 78.75 180)
+    (fp_text reference J5 (at 0 0.5) (layer F.SilkS) hide
+      (effects (font (size 1 1) (thickness 0.15)))
+    )
+    (fp_text value Conn_01x01_Female (at 0 -0.5) (layer F.Fab) hide
+      (effects (font (size 1 1) (thickness 0.15)))
+    )
+    (pad 1 smd rect (at -0.1 -2.7 180) (size 8 4) (layers F.Cu F.Mask)
+      (net 2 "Net-(J2-Pad1)"))
   )
   (module MountingHole:MountingHole_6mm_Pad_Via (layer F.Cu)
@@
     (arrow2b (pts (xy 122 43) (xy 123.126504 42.413579)))
   )
+  (via (at 123.25 82.75) (size 0.8) (drill 0.4) (layers F.Cu B.Cu) (net 1))
+  (via (at 125 82.75) (size 0.8) (drill 0.4) (layers F.Cu B.Cu) (net 1))
+  (via (at 126.5 82.75) (size 0.8) (drill 0.4) (layers F.Cu B.Cu) (net 1))
+  (via (at 128 82.75) (size 0.8) (drill 0.4) (layers F.Cu B.Cu) (net 1))
+  (via (at 129.5 82.75) (size 0.8) (drill 0.4) (layers F.Cu B.Cu) (net 1))
   (via (at 122 58) (size 2) (drill 1) (layers F.Cu B.Cu) (net 1))
   (via (at 128 64) (size 2) (drill 1) (layers F.Cu B.Cu) (net 1))
@@
   (via (at 118 60) (size 2) (drill 1) (layers F.Cu B.Cu) (net 1))
   (via (at 118 68) (size 2) (drill 1) (layers F.Cu B.Cu) (net 1))
+  (via (at 126.5 81.5) (size 0.8) (drill 0.4) (layers F.Cu B.Cu) (net 1))
+  (via (at 129.5 81.5) (size 0.8) (drill 0.4) (layers F.Cu B.Cu) (net 1))
+  (via (at 123.25 81.5) (size 0.8) (drill 0.4) (layers F.Cu B.Cu) (net 1))
+  (via (at 125 81.5) (size 0.8) (drill 0.4) (layers F.Cu B.Cu) (net 1))
+  (via (at 128 81.5) (size 0.8) (drill 0.4) (layers F.Cu B.Cu) (net 1))
+  (via (at 129.5 80.25) (size 0.8) (drill 0.4) (layers F.Cu B.Cu) (net 1))
+  (via (at 126.5 80.25) (size 0.8) (drill 0.4) (layers F.Cu B.Cu) (net 1))
+  (via (at 128 80.25) (size 0.8) (drill 0.4) (layers F.Cu B.Cu) (net 1))
+  (via (at 123.25 80.25) (size 0.8) (drill 0.4) (layers F.Cu B.Cu) (net 1))
+  (via (at 125 80.25) (size 0.8) (drill 0.4) (layers F.Cu B.Cu) (net 1))
+  (via (at 147.75 80.25) (size 0.8) (drill 0.4) (layers F.Cu B.Cu) (net 2))
+  (via (at 144.75 80.25) (size 0.8) (drill 0.4) (layers F.Cu B.Cu) (net 2))
+  (via (at 149.25 82.75) (size 0.8) (drill 0.4) (layers F.Cu B.Cu) (net 2))
+  (via (at 144.75 81.5) (size 0.8) (drill 0.4) (layers F.Cu B.Cu) (net 2))
+  (via (at 147.75 82.75) (size 0.8) (drill 0.4) (layers F.Cu B.Cu) (net 2))
+  (via (at 144.75 82.75) (size 0.8) (drill 0.4) (layers F.Cu B.Cu) (net 2))
+  (via (at 147.75 81.5) (size 0.8) (drill 0.4) (layers F.Cu B.Cu) (net 2))
+  (via (at 146.25 81.5) (size 0.8) (drill 0.4) (layers F.Cu B.Cu) (net 2))
+  (via (at 151 81.5) (size 0.8) (drill 0.4) (layers F.Cu B.Cu) (net 2))
+  (via (at 149.25 81.5) (size 0.8) (drill 0.4) (layers F.Cu B.Cu) (net 2))
+  (via (at 151 80.25) (size 0.8) (drill 0.4) (layers F.Cu B.Cu) (net 2))
+  (via (at 149.25 80.25) (size 0.8) (drill 0.4) (layers F.Cu B.Cu) (net 2))
+  (via (at 146.25 82.75) (size 0.8) (drill 0.4) (layers F.Cu B.Cu) (net 2))
+  (via (at 151 82.75) (size 0.8) (drill 0.4) (layers F.Cu B.Cu) (net 2))
+  (via (at 146.25 80.25) (size 0.8) (drill 0.4) (layers F.Cu B.Cu) (net 2))
   (via (at 152 58) (size 2) (drill 1) (layers F.Cu B.Cu) (net 2))
   (via (at 152 70) (size 2) (drill 1) (layers F.Cu B.Cu) (net 2))
