File: korad_kel103_converter.sch (KiCad schematic (older format))
At the start: 4 parts, among them J1 Conn_01x01_Female, J2 Conn_01x01_Female, J3 Conn_01x01_Female, J4 Conn_01x01_Female

Commit message: Adding readme
Parts:
- added J5, J6: Conn_01x01_Female, Local:SMD_pad_connector, symbol Connector:Conn_01x01_Female
Connections:
- net at J2.1 (Pin_1), J4.1 (Pin_1): now also J5.1 (Pin_1)
- net at J1.1 (Pin_1), J3.1 (Pin_1): now also J6.1 (Pin_1)
Changed lines of the file:
@@
+$EndComp
+$Comp
+L Connector:Conn_01x01_Female J1
+U 1 1 617A325B
+P 4275 2875
+F 0 "J1" H 4167 2650 50  0000 C CNN
+F 1 "Conn_01x01_Female" H 4167 2741 50  0000 C CNN
+F 2 "Local:electronic_load_conn" H 4275 2875 50  0001 C CNN
+F 3 "~" H 4275 2875 50  0001 C CNN
+	1    4275 2875
+	-1   0    0    1
 $EndComp
 $Comp
@@
 	-1   0    0    1
 $EndComp
+Wire Wire Line
+	4475 2875 4850 2875
+Wire Wire Line
+	4500 2500 4850 2500
 $Comp
-L Connector:Conn_01x01_Female J1
-U 1 1 617A325B
-P 4275 2875
-F 0 "J1" H 4167 2650 50  0000 C CNN
-F 1 "Conn_01x01_Female" H 4167 2741 50  0000 C CNN
-F 2 "Local:electronic_load_conn" H 4275 2875 50  0001 C CNN
-F 3 "~" H 4275 2875 50  0001 C CNN
-	1    4275 2875
-	-1   0    0    1
+L Connector:Conn_01x01_Female J5
+U 1 1 617A8E50
+P 4850 2050
+F 0 "J5" V 4788 1962 50  0000 R CNN
+F 1 "Conn_01x01_Female" V 4697 1962 50  0000 R CNN
+F 2 "Local:SMD_pad_connector" H 4850 2050 50  0001 C CNN
+F 3 "~" H 4850 2050 50  0001 C CNN
+	1    4850 2050
+	0    -1   -1   0
 $EndComp
 Wire Wire Line
-	4500 2500 4950 2500
+	4850 2250 4850 2500
+Connection ~ 4850 2500
 Wire Wire Line
-	4475 2875 4925 2875
+	4850 2500 4950 2500
+$Comp
+L Connector:Conn_01x01_Female J6
+U 1 1 617A9DA1
+P 4850 3325
+F 0 "J6" V 4696 3373 50  0000 L CNN
+F 1 "Conn_01x01_Female" V 4787 3373 50  0000 L CNN
+F 2 "Local:SMD_pad_connector" H 4850 3325 50  0001 C CNN
+F 3 "~" H 4850 3325 50  0001 C CNN
+	1    4850 3325
+	0    1    1    0
+$EndComp
+Wire Wire Line
+	4850 3125 4850 2875
+Connection ~ 4850 2875
+Wire Wire Line
+	4850 2875 4925 2875
 $EndSCHEMATC
