File: korad_kel103_converter.kicad_pcb (KiCad board)
At the start: 2 copper layers, 48 x 44.9 mm, 4 parts, among them J1 Conn_01x01_Female, J2 Conn_01x01_Female, J3 Conn_01x01_Female, J4 Conn_01x01_Female

Commit message: Adding readme
Other:
- board size 48 x 44.9 mm -> 47.9 x 44.9 mm
Changed lines of the file:
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@@
   (general
     (thickness 1.6)
-    (drawings 15)
+    (drawings 20)
     (tracks 16)
     (zones 0)
@@
     (38 B.Mask user)
     (39 F.Mask user)
-    (40 Dwgs.User user)
+    (40 Dwgs.User user hide)
     (41 Cmts.User user)
-    (42 Eco1.User user)
+    (42 Eco1.User user hide)
     (43 Eco2.User user)
     (44 Edge.Cuts user)
     (45 Margin user)
     (46 B.CrtYd user hide)
-    (47 F.CrtYd user hide)
+    (47 F.CrtYd user)
     (48 B.Fab user hide)
     (49 F.Fab user hide)
@@
     (mod_text_size 1 1)
     (mod_text_width 0.15)
-    (pad_size 11 11)
-    (pad_drill 6)
+    (pad_size 2 2)
+    (pad_drill 0.5)
     (pad_to_mask_clearance 0)
     (aux_axis_origin 0 0)
@@
       (net 1 "Net-(J1-Pad1)"))
   )
+  (gr_line (start 144.605411 58.953691) (end 144.53563 59.040422) (layer Edge.Cuts) (width 0.05))
+  (gr_arc (start 152.000002 63.99178) (end 152.000002 54.99178) (angle 102.5288077) (layer Edge.Cuts) (width 0.05))
+  (gr_arc (start 152.104703 64.068859) (end 152.000002 54.99178) (angle -55.0417592) (layer Edge.Cuts) (width 0.05))
+  (gr_arc (start 136.995297 54) (end 129.395298 58.949999) (angle -113.1619671) (layer Edge.Cuts) (width 0.05))
+  (gr_circle (center 136.986122 54) (end 141.986122 46.5) (layer Eco1.User) (width 0.15))
+  (gr_circle (center 122 64) (end 127 56.5) (layer Eco1.User) (width 0.15))
+  (gr_circle (center 152 64) (end 157 56.5) (layer Eco1.User) (width 0.15))
   (dimension 36 (width 0.15) (layer Dwgs.User)
     (gr_text "36.000 mm" (at 183.3 82 270) (layer Dwgs.User)
@@
     (arrow2b (pts (xy 187 55) (xy 187.586421 56.126504)))
   )
-  (gr_line (start 122 55) (end 152.000002 54.99178) (layer Edge.Cuts) (width 0.05))
-  (gr_arc (start 152.000002 63.99178) (end 152.000002 54.99178) (angle 102.5288077) (layer Edge.Cuts) (width 0.05))
   (gr_line (start 160.785686 65.944154) (end 155.400001 93.991779) (layer Edge.Cuts) (width 0.05))
   (gr_arc (start 148.000002 92.24178) (end 155.400001 93.991779) (angle 76.69476349) (layer Edge.Cuts) (width 0.05))
@@
   (gr_line (start 125.999999 99.85411) (end 137 99.85) (layer Edge.Cuts) (width 0.05))
   (gr_arc (start 126 92.25) (end 118.600001 93.999999) (angle -76.69476349) (layer Edge.Cuts) (width 0.05))
-  (gr_line (start 113.214316 65.952374) (end 118.600001 93.999999) (layer Edge.Cuts) (width 0.05))
-  (gr_arc (start 122 64) (end 122 55) (angle -102.5288077) (layer Edge.Cuts) (width 0.05))
+  (gr_line (start 113.254404 65.943462) (end 118.600001 93.999999) (layer Edge.Cuts) (width 0.05))
+  (gr_arc (start 122 64) (end 129.4 58.95) (angle -158.2178888) (layer Edge.Cuts) (width 0.05))
   (gr_circle (center 122 64) (end 113 64) (layer Dwgs.User) (width 0.15))
   (gr_line (start 137 43) (end 137 106) (layer Dwgs.User) (width 0.05))
@@
     (polygon
       (pts
-        (xy 133 100) (xy 120 100) (xy 111 55) (xy 131 55)
+        (xy 130.5 62) (xy 132.5 95.5) (xy 129 99) (xy 120.5 97.5) (xy 111 55)
+        (xy 127 55)
+      )
+    )
+  )
+  (zone (net 1) (net_name "Net-(J1-Pad1)") (layer B.Cu) (hatch edge 0.508)
+    (connect_pads yes (clearance 0.508))
+    (min_thickness 0.254)
+    (fill yes (arc_segments 32) (thermal_gap 0.508) (thermal_bridge_width 0.508) (smoothing fillet) (radius 8))
+    (polygon
+      (pts
+        (xy 130.5 62.008378) (xy 132.5 95.5) (xy 129 99) (xy 120.5 97.5) (xy 111 55)
+        (xy 127 55)
       )
     )
@@
     (polygon
       (pts
-        (xy 141 100) (xy 154 100) (xy 163 55) (xy 143 55)
-      )
-    )
-  )
-  (zone (net 1) (net_name "Net-(J1-Pad1)") (layer B.Cu) (hatch edge 0.508)
-    (connect_pads yes (clearance 0.508))
-    (min_thickness 0.254)
-    (fill yes (arc_segments 32) (thermal_gap 0.508) (thermal_bridge_width 0.508) (smoothing fillet) (radius 8))
-    (polygon
-      (pts
-        (xy 133 100) (xy 120 100) (xy 111 55) (xy 131 55)
+        (xy 143.805728 61.754048) (xy 141.805728 95.254048) (xy 145.305728 98.754048) (xy 153.5 97.5) (xy 163.305728 54.754048)
+        (xy 147.305728 54.754048)
       )
     )
@@
     (polygon
       (pts
-        (xy 141 100) (xy 154 100) (xy 163 55) (xy 143 55)
+        (xy 143.805728 61.753723) (xy 141.805728 95.253723) (xy 145.305728 98.753723) (xy 153.5 97.499675) (xy 163.305728 54.753723)
+        (xy 147.305728 54.753723)
       )
     )

Commit message: Creating gerbers and ordering PCB
Parts:
- added J5: Conn_01x01_Female, Local:SMD_pad_connector, F.Cu at (137.0, 93.7)
- added J6: Conn_01x01_Female, Local:SMD_pad_connector, F.Cu at (137.2, 93.5)
Routing:
- net Net-(J2-Pad1): vias 8 -> 23
- net Net-(J1-Pad1): vias 8 -> 23
Other:
- board size 47.9 x 44.9 mm -> 47.9 x 43.4 mm
